Commit message: removed d435 plug and works

File: catkin_ws/src/fmauch_universal_robot/ur_e_description/urdf/ur3e_robot_bunkier.urdf.xacro (robot description, xacro)
@@ -1,3 +1,4 @@
 <?xml version="1.0"?>
+<!-- -->
 <robot xmlns:xacro="http://ros.org/wiki/xacro"
   name="ur3e" >
@@ -6,14 +7,23 @@
   <!-- ur3e -->
   <xacro:include filename="$(find ur_e_description)/urdf/ur3e.urdf.xacro" />
-  <!-- arm -->
+  <!-- intel realsense -->
+  <xacro:include filename="$(find realsense2_description)/urdf/_d435.urdf.xacro">
+	<!--<xacro:arg name="add_plug" value="false"/>-->
+  </xacro:include>
+<!-- arm -->
   <xacro:arg name="kinematics_config" default="$(find ur_e_description)/config/ur3e_default.yaml"/>
   <xacro:ur3e_robot prefix="" joint_limited="false"
     kinematics_file="${load_yaml('$(arg kinematics_config)')}"
   />
-  <link name="world" />
-  <joint name="world_joint" type="fixed">
-    <parent link="world" />
-    <child link = "base_link" />
-    <origin xyz="0.0 0.0 0.0" rpy="0.0 0.0 0.0" />
+  <link name="d435_link">
+  </link>
+  <joint name="d435_joint" type="fixed">
+    <origin xyz="0 0 0.0" rpy="0 0 0" />
+    <parent link="tool0"/>
+    <child link="d435_link"/>
   </joint>
+  <xacro:sensor_d435 parent="d435_link" name="intel_cam" >
+    <origin xyz="0.0 0.10 0.0" rpy="1.570 -1.570 0"/>
+     <!-- <origin xyz="0.20 0 0" rpy="0 0 0"/> -->
+  </xacro:sensor_d435>
 </robot>

File: catkin_ws/src/realsense-ros/realsense2_description/urdf/_d435.urdf.xacro (robot description, xacro)
@@ -124,9 +124,4 @@
       <link name="${name}_color_optical_frame"/>
     </xacro:if>
-    <xacro:if value="$(arg add_plug)">
-      <xacro:usb_plug parent="${name}_link">
-        <origin xyz="${d435_cam_mount_from_center_offset - 0.02095} ${-d435_cam_depth_py - 0.0353} 0" rpy="0 0 0"/>
-      </xacro:usb_plug>
-    </xacro:if>
   </xacro:macro>
 </robot>

Commit message: added 3d printed part

File: catkin_ws/src/fmauch_universal_robot/ur_e_description/urdf/ur3e_robot_bunkier.urdf.xacro (robot description, xacro)
@@ -16,13 +16,38 @@
     kinematics_file="${load_yaml('$(arg kinematics_config)')}"
   />
+  <link name="connector_link">
+	<visual>
+	<origin xyz="0.0 0.0 0.0" rpy="0.0 0.0 0.0"/>
+	<geometry>
+	    <mesh filename="package://ur_e_description/meshes/3dprint/mocowanie.dae" scale="0.001 0.001 0.001"/>
+	</geometry>
+    </visual>
+    <collision>
+	<origin xyz="0.0 0.0 0.0" rpy="0.0 0.0 0.0"/>
+	<geometry>
+	    <mesh filename="package://ur_e_description/meshes/3dprint/mocowanie.stl" scale="0.001 0.001 0.001"/>
+	</geometry>
+    </collision>
+    <inertial>
+        <!-- The following are not reliable values, and should not be used for modeling -->
+        <mass value="0.1" />
+        <origin xyz="0 0 0" />
+        <inertia ixx="28265492.000000" ixy="-83622.820312" ixz="-1018.753967" iyx="-83622.820312" iyy="10976009.000000" iyz="-92508.718750" izx="-1018.753967" izy="-92508.718750" izz="39048324.000000" />
+      </inertial>
+  </link>
+  <joint name="connector_joint" type="fixed">
+    <origin xyz="0 0 0" rpy="0 0 0" />
+    <parent link="tool0"/>
+    <child link="connector_link"/>
+  </joint>
   <link name="d435_link">
   </link>
   <joint name="d435_joint" type="fixed">
     <origin xyz="0 0 0.0" rpy="0 0 0" />
-    <parent link="tool0"/>
+    <parent link="connector_link"/>
     <child link="d435_link"/>
   </joint>
   <xacro:sensor_d435 parent="d435_link" name="intel_cam" >
-    <origin xyz="0.0 0.10 0.0" rpy="1.570 -1.570 0"/>
+    <origin xyz="0.0 0.08 0.0155" rpy="1.570 -1.570 0"/>
      <!-- <origin xyz="0.20 0 0" rpy="0 0 0"/> -->
   </xacro:sensor_d435>

Commit message: removed d435 plug and works

File: catkin_ws/src/fmauch_universal_robot/ur_e_description/urdf/ur3e_robot_bunkier.urdf.xacro (robot description, xacro)
@@ -52,3 +52,28 @@
      <!-- <origin xyz="0.20 0 0" rpy="0 0 0"/> -->
   </xacro:sensor_d435>
+  <link name="gripper">
+    <visual>
+	<origin xyz="0.0 0.0 0.0" rpy="0.0 0.0 0.0"/>
+	<geometry>
+	    <mesh filename="package://ur_e_description/meshes/rg2_gripper/rg2_.stl" scale="0.001 0.001 0.001"/>
+	</geometry>
+    </visual>
+    <collision>
+	<origin xyz="0.0 0.0 0.0" rpy="0.0 0.0 0.0"/>
+	<geometry>
+	    <mesh filename="package://ur_e_description/meshes/rg2_gripper/rg2_.stl" scale="0.001 0.001 0.001"/>
+	</geometry>
+    </collision>
+    <inertial>
+        <!-- The following are not reliable values, and should not be used for modeling -->
+        <mass value="0.1" />
+        <origin xyz="0 0 0" />
+        <inertia ixx="575346816.000000" ixy="26432.207031" ixz="27110.214844" iyx="26432.207031" iyy="640683008.000000" iyz="143325.546875" izx="27110.214844" izy="143325.546875" izz="116270144.000000" />
+      </inertial>
+  </link>
+  <joint name="gripper_joint" type="fixed">
+    <origin xyz="0 0.009 0.055" rpy="0 0 0"/>
+    <parent link="connector_link"/>
+    <child link="gripper"/>
+  </joint>
 </robot>

Commit message: correct orientation and efficency

File: catkin_ws/src/fmauch_universal_robot/ur_e_description/urdf/ur3e_robot_bunkier.urdf.xacro (robot description, xacro)
@@ -50,6 +50,14 @@
   <xacro:sensor_d435 parent="d435_link" name="intel_cam" >
     <origin xyz="0.0 0.08 0.0155" rpy="1.570 -1.570 0"/>
-     <!-- <origin xyz="0.20 0 0" rpy="0 0 0"/> -->
+     <!-- <origin xyz="0.0 0.08 0.0155" rpy="0 0 0"/> -->
   </xacro:sensor_d435>
+  <link name="dumb_link">
+    <origin xyz="0.0 0.0 0.0" rpy="0 0 0"/>
+  </link>
+  <joint name="dumb_joint" type="fixed">
+    <origin xyz="0 0 0.0" rpy="1.57 0 3.14" />
+    <parent link="d435_link"/>
+    <child link="dumb_link"/>
+  </joint>
   <link name="gripper">
     <visual>

Commit message: aruco on pcl works, but needs calibration for d435 rgb cam

File: catkin_ws/src/fmauch_universal_robot/ur_e_description/urdf/ur3e_robot_bunkier.urdf.xacro (robot description, xacro)
@@ -60,4 +60,12 @@
     <child link="dumb_link"/>
   </joint>
+  <link name="dumb_link_2">
+    <origin xyz="0.0 0.08 0.0155" rpy="0 0 0"/>
+  </link>
+  <joint name="dumb_joint_2" type="fixed">
+    <origin xyz="0 0 0.0" rpy="-1.57 0.0 0.0" />
+    <parent link="dumb_link"/>
+    <child link="dumb_link_2"/>
+  </joint>
   <link name="gripper">
     <visual>
